File: Mechanical-PicoBoard-W/Mechanical-PicoBoard-W.kicad_sch (KiCad schematic)
At the start: 0 parts

Commit message: recovery day
Parts:
- added A1: RaspberryPi_Pico_W, Library:RaspberryPi_Pico_Common_THT_Model, symbol MCU_Module:RaspberryPi_Pico_W
- added BT1: Battery_Cell, Battery:BatteryHolder_Keystone_1042_1x18650, symbol Device:Battery_Cell
- added D1: esc, Diode_THT:D_DO-35_SOD27_P7.62mm_Horizontal, symbol Diode:1N4148
- added D10: 9, Diode_THT:D_DO-35_SOD27_P7.62mm_Horizontal, symbol Diode:1N4148
- added D11: 0, Diode_THT:D_DO-35_SOD27_P7.62mm_Horizontal, symbol Diode:1N4148
- added D12: -, Diode_THT:D_DO-35_SOD27_P7.62mm_Horizontal, symbol Diode:1N4148
- added D13: =, Diode_THT:D_DO-35_SOD27_P7.62mm_Horizontal, symbol Diode:1N4148
- added D14: Backspace, Diode_THT:D_DO-35_SOD27_P7.62mm_Horizontal, symbol Diode:1N4148
- added D15: del, Diode_THT:D_DO-35_SOD27_P7.62mm_Horizontal, symbol Diode:1N4148
- added D16: tab, Diode_THT:D_DO-35_SOD27_P7.62mm_Horizontal, symbol Diode:1N4148
- added D17: Q, Diode_THT:D_DO-35_SOD27_P7.62mm_Horizontal, symbol Diode:1N4148
- added D18: W, Diode_THT:D_DO-35_SOD27_P7.62mm_Horizontal, symbol Diode:1N4148
- added D19: E, Diode_THT:D_DO-35_SOD27_P7.62mm_Horizontal, symbol Diode:1N4148
- added D2: 1, Diode_THT:D_DO-35_SOD27_P7.62mm_Horizontal, symbol Diode:1N4148
- added D20: R, Diode_THT:D_DO-35_SOD27_P7.62mm_Horizontal, symbol Diode:1N4148
- added D21: T, Diode_THT:D_DO-35_SOD27_P7.62mm_Horizontal, symbol Diode:1N4148
- added D22: Y, Diode_THT:D_DO-35_SOD27_P7.62mm_Horizontal, symbol Diode:1N4148
- added D23: U, Diode_THT:D_DO-35_SOD27_P7.62mm_Horizontal, symbol Diode:1N4148
- added D24: I, Diode_THT:D_DO-35_SOD27_P7.62mm_Horizontal, symbol Diode:1N4148
- added D25: O, Diode_THT:D_DO-35_SOD27_P7.62mm_Horizontal, symbol Diode:1N4148
- added D26: P, Diode_THT:D_DO-35_SOD27_P7.62mm_Horizontal, symbol Diode:1N4148
- added D27: [, Diode_THT:D_DO-35_SOD27_P7.62mm_Horizontal, symbol Diode:1N4148
- added D28: ], Diode_THT:D_DO-35_SOD27_P7.62mm_Horizontal, symbol Diode:1N4148
- added D29: \, Diode_THT:D_DO-35_SOD27_P7.62mm_Horizontal, symbol Diode:1N4148
- added D3: 2, Diode_THT:D_DO-35_SOD27_P7.62mm_Horizontal, symbol Diode:1N4148
- added D30: home, Diode_THT:D_DO-35_SOD27_P7.62mm_Horizontal, symbol Diode:1N4148
- added D31: caps lock, Diode_THT:D_DO-35_SOD27_P7.62mm_Horizontal, symbol Diode:1N4148
- added D32: A, Diode_THT:D_DO-35_SOD27_P7.62mm_Horizontal, symbol Diode:1N4148
- added D33: S, Diode_THT:D_DO-35_SOD27_P7.62mm_Horizontal, symbol Diode:1N4148
- added D34: D, Diode_THT:D_DO-35_SOD27_P7.62mm_Horizontal, symbol Diode:1N4148
- added D35: F, Diode_THT:D_DO-35_SOD27_P7.62mm_Horizontal, symbol Diode:1N4148
- added D36: G, Diode_THT:D_DO-35_SOD27_P7.62mm_Horizontal, symbol Diode:1N4148
- added D37: H, Diode_THT:D_DO-35_SOD27_P7.62mm_Horizontal, symbol Diode:1N4148
- added D38: J, Diode_THT:D_DO-35_SOD27_P7.62mm_Horizontal, symbol Diode:1N4148
- added D39: K, Diode_THT:D_DO-35_SOD27_P7.62mm_Horizontal, symbol Diode:1N4148
- added D4: 3, Diode_THT:D_DO-35_SOD27_P7.62mm_Horizontal, symbol Diode:1N4148
- added D40: L, Diode_THT:D_DO-35_SOD27_P7.62mm_Horizontal, symbol Diode:1N4148
- added D41: ;, Diode_THT:D_DO-35_SOD27_P7.62mm_Horizontal, symbol Diode:1N4148
- added D42: ', Diode_THT:D_DO-35_SOD27_P7.62mm_Horizontal, symbol Diode:1N4148
- added D43: enter, Diode_THT:D_DO-35_SOD27_P7.62mm_Horizontal, symbol Diode:1N4148
- added D44: page up, Diode_THT:D_DO-35_SOD27_P7.62mm_Horizontal, symbol Diode:1N4148
- added D45, D56: shift, Diode_THT:D_DO-35_SOD27_P7.62mm_Horizontal, symbol Diode:1N4148
- added D46: Z, Diode_THT:D_DO-35_SOD27_P7.62mm_Horizontal, symbol Diode:1N4148
- added D47: X, Diode_THT:D_DO-35_SOD27_P7.62mm_Horizontal, symbol Diode:1N4148
- added D48: C, Diode_THT:D_DO-35_SOD27_P7.62mm_Horizontal, symbol Diode:1N4148
- added D49: V, Diode_THT:D_DO-35_SOD27_P7.62mm_Horizontal, symbol Diode:1N4148
- added D5: 4, Diode_THT:D_DO-35_SOD27_P7.62mm_Horizontal, symbol Diode:1N4148
- added D50: B, Diode_THT:D_DO-35_SOD27_P7.62mm_Horizontal, symbol Diode:1N4148
- added D51: N, Diode_THT:D_DO-35_SOD27_P7.62mm_Horizontal, symbol Diode:1N4148
- added D52: M, Diode_THT:D_DO-35_SOD27_P7.62mm_Horizontal, symbol Diode:1N4148
- added D53: ,, Diode_THT:D_DO-35_SOD27_P7.62mm_Horizontal, symbol Diode:1N4148
- added D54: ., Diode_THT:D_DO-35_SOD27_P7.62mm_Horizontal, symbol Diode:1N4148
- added D55: /, Diode_THT:D_DO-35_SOD27_P7.62mm_Horizontal, symbol Diode:1N4148
- added D57: up, Diode_THT:D_DO-35_SOD27_P7.62mm_Horizontal, symbol Diode:1N4148
- added D58: page down, Diode_THT:D_DO-35_SOD27_P7.62mm_Horizontal, symbol Diode:1N4148
- added D59: ctrl, Diode_THT:D_DO-35_SOD27_P7.62mm_Horizontal, symbol Diode:1N4148
- added D6: 5, Diode_THT:D_DO-35_SOD27_P7.62mm_Horizontal, symbol Diode:1N4148
- added D60, D65: alt, Diode_THT:D_DO-35_SOD27_P7.62mm_Horizontal, symbol Diode:1N4148
- added D61: gui, Diode_THT:D_DO-35_SOD27_P7.62mm_Horizontal, symbol Diode:1N4148
- added D62, D64: space, Diode_THT:D_DO-35_SOD27_P7.62mm_Horizontal, symbol Diode:1N4148
- added D63: func, Diode_THT:D_DO-35_SOD27_P7.62mm_Horizontal, symbol Diode:1N4148
- added D66: left, Diode_THT:D_DO-35_SOD27_P7.62mm_Horizontal, symbol Diode:1N4148
- added D67: down, Diode_THT:D_DO-35_SOD27_P7.62mm_Horizontal, symbol Diode:1N4148
- added D68: right, Diode_THT:D_DO-35_SOD27_P7.62mm_Horizontal, symbol Diode:1N4148
- added D7: 6, Diode_THT:D_DO-35_SOD27_P7.62mm_Horizontal, symbol Diode:1N4148
- added D8: 7, Diode_THT:D_DO-35_SOD27_P7.62mm_Horizontal, symbol Diode:1N4148
- added D9: 8, Diode_THT:D_DO-35_SOD27_P7.62mm_Horizontal, symbol Diode:1N4148
- added SW1: esc, Button_Switch_Keyboard:SW_Cherry_MX_1.00u_PCB, symbol Switch:SW_Push_45deg
- added SW10: 9, Button_Switch_Keyboard:SW_Cherry_MX_1.00u_PCB, symbol Switch:SW_Push_45deg
- added SW11: 0, Button_Switch_Keyboard:SW_Cherry_MX_1.00u_PCB, symbol Switch:SW_Push_45deg
- added SW12: -, Button_Switch_Keyboard:SW_Cherry_MX_1.00u_PCB, symbol Switch:SW_Push_45deg
- added SW13: =, Button_Switch_Keyboard:SW_Cherry_MX_1.00u_PCB, symbol Switch:SW_Push_45deg
- added SW14: Backspace, Button_Switch_Keyboard:SW_Cherry_MX_2.00u_PCB, symbol Switch:SW_Push_45deg
- added SW15: del, Button_Switch_Keyboard:SW_Cherry_MX_1.00u_PCB, symbol Switch:SW_Push_45deg
- added SW16: tab, Button_Switch_Keyboard:SW_Cherry_MX_1.50u_PCB, symbol Switch:SW_Push_45deg
- added SW17: Q, Button_Switch_Keyboard:SW_Cherry_MX_1.00u_PCB, symbol Switch:SW_Push_45deg
- added SW18: W, Button_Switch_Keyboard:SW_Cherry_MX_1.00u_PCB, symbol Switch:SW_Push_45deg
- added SW19: E, Button_Switch_Keyboard:SW_Cherry_MX_1.00u_PCB, symbol Switch:SW_Push_45deg
- added SW2: 1, Button_Switch_Keyboard:SW_Cherry_MX_1.00u_PCB, symbol Switch:SW_Push_45deg
- added SW20: R, Button_Switch_Keyboard:SW_Cherry_MX_1.00u_PCB, symbol Switch:SW_Push_45deg
- added SW21: T, Button_Switch_Keyboard:SW_Cherry_MX_1.00u_PCB, symbol Switch:SW_Push_45deg
- added SW22: Y, Button_Switch_Keyboard:SW_Cherry_MX_1.00u_PCB, symbol Switch:SW_Push_45deg
- added SW23: U, Button_Switch_Keyboard:SW_Cherry_MX_1.00u_PCB, symbol Switch:SW_Push_45deg
- added SW24: I, Button_Switch_Keyboard:SW_Cherry_MX_1.00u_PCB, symbol Switch:SW_Push_45deg
- added SW25: O, Button_Switch_Keyboard:SW_Cherry_MX_1.00u_PCB, symbol Switch:SW_Push_45deg
- added SW26: P, Button_Switch_Keyboard:SW_Cherry_MX_1.00u_PCB, symbol Switch:SW_Push_45deg
- added SW27: [, Button_Switch_Keyboard:SW_Cherry_MX_1.00u_PCB, symbol Switch:SW_Push_45deg
- added SW28: ], Button_Switch_Keyboard:SW_Cherry_MX_1.00u_PCB, symbol Switch:SW_Push_45deg
- added SW29: \, Button_Switch_Keyboard:SW_Cherry_MX_1.50u_PCB, symbol Switch:SW_Push_45deg
- added SW3: 2, Button_Switch_Keyboard:SW_Cherry_MX_1.00u_PCB, symbol Switch:SW_Push_45deg
- added SW30: home, Button_Switch_Keyboard:SW_Cherry_MX_1.00u_PCB, symbol Switch:SW_Push_45deg
- added SW31: caps lock, Button_Switch_Keyboard:SW_Cherry_MX_1.75u_PCB, symbol Switch:SW_Push_45deg
- added SW32: A, Button_Switch_Keyboard:SW_Cherry_MX_1.00u_PCB, symbol Switch:SW_Push_45deg
- added SW33: S, Button_Switch_Keyboard:SW_Cherry_MX_1.00u_PCB, symbol Switch:SW_Push_45deg
- added SW34: D, Button_Switch_Keyboard:SW_Cherry_MX_1.00u_PCB, symbol Switch:SW_Push_45deg
- added SW35: F, Button_Switch_Keyboard:SW_Cherry_MX_1.00u_PCB, symbol Switch:SW_Push_45deg
- added SW36: G, Button_Switch_Keyboard:SW_Cherry_MX_1.00u_PCB, symbol Switch:SW_Push_45deg
- added SW37: H, Button_Switch_Keyboard:SW_Cherry_MX_1.00u_PCB, symbol Switch:SW_Push_45deg
- added SW38: J, Button_Switch_Keyboard:SW_Cherry_MX_1.00u_PCB, symbol Switch:SW_Push_45deg
- added SW39: K, Button_Switch_Keyboard:SW_Cherry_MX_1.00u_PCB, symbol Switch:SW_Push_45deg
- added SW4: 3, Button_Switch_Keyboard:SW_Cherry_MX_1.00u_PCB, symbol Switch:SW_Push_45deg
- added SW40: L, Button_Switch_Keyboard:SW_Cherry_MX_1.00u_PCB, symbol Switch:SW_Push_45deg
- added SW41: ;, Button_Switch_Keyboard:SW_Cherry_MX_1.00u_PCB, symbol Switch:SW_Push_45deg
- added SW42: ', Button_Switch_Keyboard:SW_Cherry_MX_1.00u_PCB, symbol Switch:SW_Push_45deg
- added SW43: enter, Button_Switch_Keyboard:SW_Cherry_MX_2.25u_PCB, symbol Switch:SW_Push_45deg
- added SW44: page up, Button_Switch_Keyboard:SW_Cherry_MX_1.00u_PCB, symbol Switch:SW_Push_45deg
- added SW45: shift, Button_Switch_Keyboard:SW_Cherry_MX_2.25u_PCB, symbol Switch:SW_Push_45deg
- added SW46: Z, Button_Switch_Keyboard:SW_Cherry_MX_1.00u_PCB, symbol Switch:SW_Push_45deg
- added SW47: X, Button_Switch_Keyboard:SW_Cherry_MX_1.00u_PCB, symbol Switch:SW_Push_45deg
- added SW48: C, Button_Switch_Keyboard:SW_Cherry_MX_1.00u_PCB, symbol Switch:SW_Push_45deg
- added SW49: V, Button_Switch_Keyboard:SW_Cherry_MX_1.00u_PCB, symbol Switch:SW_Push_45deg
- added SW5: 4, Button_Switch_Keyboard:SW_Cherry_MX_1.00u_PCB, symbol Switch:SW_Push_45deg
- added SW50: B, Button_Switch_Keyboard:SW_Cherry_MX_1.00u_PCB, symbol Switch:SW_Push_45deg
- added SW51: N, Button_Switch_Keyboard:SW_Cherry_MX_1.00u_PCB, symbol Switch:SW_Push_45deg
- added SW52: M, Button_Switch_Keyboard:SW_Cherry_MX_1.00u_PCB, symbol Switch:SW_Push_45deg
- added SW53: ,, Button_Switch_Keyboard:SW_Cherry_MX_1.00u_PCB, symbol Switch:SW_Push_45deg
- added SW54: ., Button_Switch_Keyboard:SW_Cherry_MX_1.00u_PCB, symbol Switch:SW_Push_45deg
- added SW55: /, Button_Switch_Keyboard:SW_Cherry_MX_1.00u_PCB, symbol Switch:SW_Push_45deg
- added SW56: shift, Button_Switch_Keyboard:SW_Cherry_MX_1.75u_PCB, symbol Switch:SW_Push_45deg
- added SW57: up, Button_Switch_Keyboard:SW_Cherry_MX_1.00u_PCB, symbol Switch:SW_Push_45deg
- added SW58: page down, Button_Switch_Keyboard:SW_Cherry_MX_1.00u_PCB, symbol Switch:SW_Push_45deg
- added SW59: ctrl, Button_Switch_Keyboard:SW_Cherry_MX_1.25u_PCB, symbol Switch:SW_Push_45deg
- added SW6: 5, Button_Switch_Keyboard:SW_Cherry_MX_1.00u_PCB, symbol Switch:SW_Push_45deg
- added SW60: alt, Button_Switch_Keyboard:SW_Cherry_MX_1.25u_PCB, symbol Switch:SW_Push_45deg
- added SW61: gui, Button_Switch_Keyboard:SW_Cherry_MX_1.25u_PCB, symbol Switch:SW_Push_45deg
- added SW62, SW64: space, Button_Switch_Keyboard:SW_Cherry_MX_2.25u_PCB, symbol Switch:SW_Push_45deg
- added SW63: func, Button_Switch_Keyboard:SW_Cherry_MX_1.75u_PCB, symbol Switch:SW_Push_45deg
- added SW65: alt, Button_Switch_Keyboard:SW_Cherry_MX_1.00u_PCB, symbol Switch:SW_Push_45deg
- added SW66: left, Button_Switch_Keyboard:SW_Cherry_MX_1.00u_PCB, symbol Switch:SW_Push_45deg
- added SW67: down, Button_Switch_Keyboard:SW_Cherry_MX_1.00u_PCB, symbol Switch:SW_Push_45deg
- added SW68: right, Button_Switch_Keyboard:SW_Cherry_MX_1.00u_PCB, symbol Switch:SW_Push_45deg
- added SW69: RotaryEncoder_Switch, Library:RotaryEncoder_Alps_EC11E-Switch_Vertical_H20mm_Model, symbol Device:RotaryEncoder_Switch
- added SW7: 6, Button_Switch_Keyboard:SW_Cherry_MX_1.00u_PCB, symbol Switch:SW_Push_45deg
- added SW8: 7, Button_Switch_Keyboard:SW_Cherry_MX_1.00u_PCB, symbol Switch:SW_Push_45deg
- added SW9: 8, Button_Switch_Keyboard:SW_Cherry_MX_1.00u_PCB, symbol Switch:SW_Push_45deg
Connections:
- new net: D42.2 (A), SW42.1
- new net: D25.2 (A), SW25.1
- new net: D60.2 (A), SW60.1
- new net: D5.2 (A), SW5.1
- new net: D45.2 (A), SW45.1
- new net: D15.2 (A), SW15.1
- new net: D4.2 (A), SW4.1
- new net: D35.2 (A), SW35.1
- new net: D65.2 (A), SW65.1
- new net: D32.2 (A), SW32.1
- new net: D54.2 (A), SW54.1
- new net: D14.2 (A), SW14.1
- new net: D34.2 (A), SW34.1
- new net: D61.2 (A), SW61.1
- new net: D28.2 (A), SW28.1
- new net: D11.2 (A), SW11.1
- new net: D53.2 (A), SW53.1
- new net: D19.2 (A), SW19.1
- new net: D27.2 (A), SW27.1
- new net: D52.2 (A), SW52.1
- new net: D58.2 (A), SW58.1
- new net: D51.2 (A), SW51.1
- new net: D6.2 (A), SW6.1
- new net: A1.21 (GPIO16), SW69.A
- new net: A1.22 (GPIO17), SW69.B
- new net: A1.13 (GND), A1.18 (GND), A1.23 (GND), A1.28 (GND), A1.3 (GND), A1.38 (GND), A1.8 (GND), BT1.2 (-), SW69.C, SW69.S1
- new net: A1.1 (GPIO0), SW69.S2
- new net: D55.2 (A), SW55.1
- new net: D17.2 (A), SW17.1
- new net: D13.2 (A), SW13.1
- new net: D41.2 (A), SW41.1
- new net: D46.2 (A), SW46.1
- new net: D68.2 (A), SW68.1
- new net: D33.2 (A), SW33.1
- new net: D63.2 (A), SW63.1
- new net: D48.2 (A), SW48.1
- new net: D40.2 (A), SW40.1
- new net: D1.2 (A), SW1.1
- new net: D9.2 (A), SW9.1
- new net: D59.2 (A), SW59.1
- new net: D36.2 (A), SW36.1
- new net: D26.2 (A), SW26.1
- new net: D38.2 (A), SW38.1
- new net: A1.39 (VSYS), BT1.1 (+)
- new net: D39.2 (A), SW39.1
- new net: D56.2 (A), SW56.1
- new net: D18.2 (A), SW18.1
- new net: D22.2 (A), SW22.1
- new net: D50.2 (A), SW50.1
- new net: D66.2 (A), SW66.1
- new net: D3.2 (A), SW3.1
- new net: D31.2 (A), SW31.1
- new net: D47.2 (A), SW47.1
- new net: D10.2 (A), SW10.1
- new net: D57.2 (A), SW57.1
- new net: D64.2 (A), SW64.1
- new net: D16.2 (A), SW16.1
- new net: D43.2 (A), SW43.1
- new net: D44.2 (A), SW44.1
- new net: D49.2 (A), SW49.1
- new net: D21.2 (A), SW21.1
- new net: D24.2 (A), SW24.1
- new net: D23.2 (A), SW23.1
- new net: D2.2 (A), SW2.1
- new net: D8.2 (A), SW8.1
- new net: D37.2 (A), SW37.1
- new net: D29.2 (A), SW29.1
- new net: D62.2 (A), SW62.1
- new net: D20.2 (A), SW20.1
- new net: D67.2 (A), SW67.1
- new net: D30.2 (A), SW30.1
- new net: D7.2 (A), SW7.1
- new net: D12.2 (A), SW12.1
- new net Col1: A1.2 (GPIO1), SW1.2, SW16.2, SW31.2, SW45.2, SW59.2
- new net Col10: A1.14 (GPIO10), SW10.2, SW25.2, SW39.2, SW53.2
- new net Col11: A1.15 (GPIO11), SW11.2, SW26.2, SW40.2, SW54.2, SW65.2
- new net Col12: A1.16 (GPIO12), SW12.2, SW27.2, SW41.2, SW55.2
- new net Col13: A1.17 (GPIO13), SW13.2, SW28.2, SW42.2, SW56.2, SW66.2
- new net Col14: A1.19 (GPIO14), SW14.2, SW29.2, SW43.2, SW57.2, SW67.2
- new net Col15: A1.20 (GPIO15), SW15.2, SW30.2, SW44.2, SW58.2, SW68.2
- new net Col2: A1.4 (GPIO2), SW17.2, SW2.2, SW60.2
- new net Col3: A1.5 (GPIO3), SW18.2, SW3.2, SW32.2, SW46.2, SW61.2
- new net Col4: A1.6 (GPIO4), SW19.2, SW33.2, SW4.2, SW47.2
- new net Col5: A1.7 (GPIO5), SW20.2, SW34.2, SW48.2, SW5.2, SW62.2
- new net Col6: A1.9 (GPIO6), SW21.2, SW35.2, SW49.2, SW6.2
- new net Col7: A1.10 (GPIO7), SW22.2, SW36.2, SW50.2, SW63.2, SW7.2
- new net Col8: A1.11 (GPIO8), SW23.2, SW37.2, SW51.2, SW8.2
- new net Col9: A1.12 (GPIO9), SW24.2, SW38.2, SW52.2, SW64.2, SW9.2
- new net Row1: A1.29 (GPIO22), D1.1 (K), D10.1 (K), D11.1 (K), D12.1 (K), D13.1 (K), D14.1 (K), D15.1 (K), D2.1 (K), D3.1 (K), D4.1 (K), D5.1 (K), D6.1 (K), D7.1 (K), D8.1 (K), D9.1 (K)
- new net Row2: A1.27 (GPIO21), D16.1 (K), D17.1 (K), D18.1 (K), D19.1 (K), D20.1 (K), D21.1 (K), D22.1 (K), D23.1 (K), D24.1 (K), D25.1 (K), D26.1 (K), D27.1 (K), D28.1 (K), D29.1 (K), D30.1 (K)
- new net Row3: A1.26 (GPIO20), D31.1 (K), D32.1 (K), D33.1 (K), D34.1 (K), D35.1 (K), D36.1 (K), D37.1 (K), D38.1 (K), D39.1 (K), D40.1 (K), D41.1 (K), D42.1 (K), D43.1 (K), D44.1 (K)
- new net Row4: A1.25 (GPIO19), D45.1 (K), D46.1 (K), D47.1 (K), D48.1 (K), D49.1 (K), D50.1 (K), D51.1 (K), D52.1 (K), D53.1 (K), D54.1 (K), D55.1 (K), D56.1 (K), D57.1 (K), D58.1 (K)
- new net Row5: A1.24 (GPIO18), D59.1 (K), D60.1 (K), D61.1 (K), D62.1 (K), D63.1 (K), D64.1 (K), D65.1 (K), D66.1 (K), D67.1 (K), D68.1 (K)
