File: Mechanical-PicoBoard-W/Mechanical-PicoBoard-W.kicad_pcb (KiCad board)
At the start: 2 copper layers, 312 x 128 mm, 139 parts, among them SW1 esc, SW10 9, SW11 0, SW12 -, SW13 =, SW14 Backspace, SW15 del, SW16 tab, SW17 Q, SW18 W, SW19 E, SW2 1, SW20 R, SW21 T, SW22 Y, SW23 U, SW24 I, SW25 O, SW26 P, SW27 [, SW28 ], SW29 \, SW3 2, SW30 home, SW31 caps lock, SW32 A, SW33 S, SW34 D, SW35 F, SW36 G, SW37 H, SW38 J, SW39 K, SW4 3, SW40 L, SW41 ;, SW42 ', SW43 enter, SW44 page up, SW45 shift, SW46 Z, SW47 X, SW48 C, SW49 V, SW5 4, SW50 B, SW51 N, SW52 M, SW53 ,, SW54 ., SW55 /, SW56 shift, SW57 up, SW58 page down, SW59 ctrl, SW6 5, SW60 alt, SW61 gui, SW62 space, SW63 func, SW64 space, SW65 alt, SW66 left, SW67 down, SW68 right, SW69 RotaryEncoder_Switch, SW7 6, SW8 7, SW9 8

Commit message: Finished
Parts:
- added G***: LOGO, abc:c, F.Cu at (249.2, 27.2)
- added G***: LOGO, abc:b, B.Cu at (170.4, 74.0)
- SW1, SW10, SW11, SW12, SW13, SW15, SW17, SW18, SW19, SW2, SW20, SW21, SW22, SW23, SW24, SW25, SW26, SW27, SW28, SW3, SW30, SW32, SW33, SW34, SW35, SW36, SW37, SW38, SW39, SW4, SW40, SW41, SW42, SW44, SW46, SW47, SW48, SW49, SW5, SW50, SW51, SW52, SW53, SW54, SW55, SW57, SW58, SW6, SW65, SW66, SW67, SW68, SW7, SW8, SW9: footprint Library:SW_Cherry_MX_1.00u_PCB_Model -> Button_Switch_Keyboard:SW_Cherry_MX_1.00u_PCB
- SW14: footprint Library:SW_Cherry_MX_2.00u_PCB_Model -> Button_Switch_Keyboard:SW_Cherry_MX_2.00u_PCB
- SW16, SW29: footprint Library:SW_Cherry_MX_1.50u_PCB_Model -> Button_Switch_Keyboard:SW_Cherry_MX_1.50u_PCB
- SW31, SW56, SW63: footprint Library:SW_Cherry_MX_1.75u_PCB_Model -> Button_Switch_Keyboard:SW_Cherry_MX_1.75u_PCB
- SW43, SW45, SW62, SW64: footprint Library:SW_Cherry_MX_2.25u_PCB_Model -> Button_Switch_Keyboard:SW_Cherry_MX_2.25u_PCB
- SW59, SW60, SW61: footprint Library:SW_Cherry_MX_1.25u_PCB_Model -> Button_Switch_Keyboard:SW_Cherry_MX_1.25u_PCB
Other:
- board text added: "FMG9167"
